Commit message: added config for downdraft

File: trossen_arm_moveit/config/wxai.srdf.xacro (robot description, xacro)
@@ -5,4 +5,8 @@
 -->
 <robot name="wxai" xmlns:xacro="http://ros.org/wiki/xacro">
+    <xacro:arg name="use_downdraft" default="true"/>
+    <xacro:property name="srdf_use_downdraft" value="$(arg use_downdraft)"/>
+    <xacro:arg name="prefix" default=""/>
+    <xacro:property name="tf_prefix" value="$(arg prefix)"/>
     <xacro:arg name="variant" default="base"/>        <!-- 'base', 'follower' -->
     <xacro:property name="arm_variant" value="$(arg variant)"/>
@@ -12,87 +16,667 @@
     <!--CHAINS: When a chain is specified, all the links along the chain (including endpoints) are included in the group. Additionally, all the joints that are parents to included links are also included. This means that joints along the chain and the parent joint of the base link are included in the group-->
     <!--SUBGROUPS: Groups can also be formed by referencing to already defined group names-->
+    <xacro:if value="${srdf_use_downdraft}">
+        <virtual_joint name="world_to_robot"
+                       type="fixed"
+                       parent_frame="world"
+                       child_link="${tf_prefix}Bottom_Box"/>
+    </xacro:if>
+    <xacro:unless value="${srdf_use_downdraft}">
+        <virtual_joint name="world_to_robot"
+                       type="fixed"
+                       parent_frame="world"
+                       child_link="${tf_prefix}base_link"/>
+    </xacro:unless>
     <group name="arm">
-        <chain base_link="base_link" tip_link="ee_gripper_link"/>
+        <chain base_link="${tf_prefix}base_link" tip_link="${tf_prefix}ee_gripper_link"/>
     </group>
     <group name="gripper">
-        <link name="carriage_left" />
-        <link name="carriage_right" />
-        <link name="gripper_left" />
-        <link name="gripper_right" />
-        <joint name="left_carriage_joint"/>
-        <passive_joint name="right_carriage_joint"/>
+        <xacro:if value="${srdf_use_downdraft}">
+            <joint name="${tf_prefix}base_and_suction"/>
+            <joint name="${tf_prefix}pillar_1_and_base_mount"/>
+            <joint name="${tf_prefix}suction_mount_and_pillar_1"/>
+            <joint name="${tf_prefix}pillar_2_and_suction_mount"/>
+            <joint name="${tf_prefix}pillar_3_and_suction_mount"/>
+            <joint name="${tf_prefix}suction_cup_and_suction_mount"/>
+            <joint name="${tf_prefix}tube_and_suction_cup"/>
+            <joint name="${tf_prefix}pillar_4_and_base_mount"/>
+        </xacro:if>
+        <joint name="${tf_prefix}ee_gripper"/>
+        <joint name="${tf_prefix}left_carriage_joint"/>
+        <joint name="${tf_prefix}left_gripper_joint"/>
+        <joint name="${tf_prefix}right_carriage_joint"/>
+        <joint name="${tf_prefix}right_gripper_joint"/>
     </group>
     <!--GROUP STATES: Purpose: Define a named state for a particular group, in terms of joint values. This is useful to define states like 'folded arms'-->
     <group_state name="sleep" group="arm">
-        <joint name="joint_0" value="0"/>
-        <joint name="joint_1" value="0"/>
-        <joint name="joint_2" value="0"/>
-        <joint name="joint_3" value="0"/>
-        <joint name="joint_4" value="0"/>
-        <joint name="joint_5" value="0"/>
+        <joint name="${tf_prefix}joint_0" value="0"/>
+        <joint name="${tf_prefix}joint_1" value="0.8"/>
+        <joint name="${tf_prefix}joint_2" value="0.8"/>
+        <joint name="${tf_prefix}joint_3" value="0"/>
+        <joint name="${tf_prefix}joint_4" value="0"/>
+        <joint name="${tf_prefix}joint_5" value="0"/>
     </group_state>
     <group_state name="upright" group="arm">
-        <joint name="joint_0" value="0"/>
-        <joint name="joint_1" value="1.5708"/>
-        <joint name="joint_2" value="1.5708"/>
-        <joint name="joint_3" value="0"/>
-        <joint name="joint_4" value="0"/>
-        <joint name="joint_5" value="0"/>
+        <joint name="${tf_prefix}joint_0" value="0"/>
+        <joint name="${tf_prefix}joint_1" value="1.5708"/>
+        <joint name="${tf_prefix}joint_2" value="1.5708"/>
+        <joint name="${tf_prefix}joint_3" value="0"/>
+        <joint name="${tf_prefix}joint_4" value="0"/>
+        <joint name="${tf_prefix}joint_5" value="0"/>
     </group_state>
     <group_state name="ready" group="arm">
-        <joint name="joint_0" value="0"/>
-        <joint name="joint_1" value="1.04719755"/>  <!-- pi / 3-->
-        <joint name="joint_2" value="0.523598776"/>  <!-- pi / 6-->
-        <joint name="joint_3" value="0.628318531"/>  <!-- pi / 5-->
-        <joint name="joint_4" value="0"/>
-        <joint name="joint_5" value="0"/>
+        <joint name="${tf_prefix}joint_0" value="0"/>
+        <joint name="${tf_prefix}joint_1" value="1.04719755"/>  <!-- pi / 3-->
+        <joint name="${tf_prefix}joint_2" value="0.523598776"/>  <!-- pi / 6-->
+        <joint name="${tf_prefix}joint_3" value="0.628318531"/>  <!-- pi / 5-->
+        <joint name="${tf_prefix}joint_4" value="0"/>
+        <joint name="${tf_prefix}joint_5" value="0"/>
     </group_state>
     <group_state name="close" group="gripper">
-        <joint name="left_carriage_joint" value="0.0"/>
-        <joint name="right_carriage_joint" value="0.0"/>
+        <joint name="${tf_prefix}left_carriage_joint" value="0.0"/>
+        <joint name="${tf_prefix}right_carriage_joint" value="0.0"/>
     </group_state>
     <group_state name="open" group="gripper">
-        <joint name="left_carriage_joint" value="0.044"/>
-        <joint name="right_carriage_joint" value="0.044"/>
+        <joint name="${tf_prefix}left_carriage_joint" value="0.044"/>
+        <joint name="${tf_prefix}right_carriage_joint" value="0.044"/>
     </group_state>
     <!--END EFFECTOR: Purpose: Represent information about an end effector.-->
-    <end_effector name="gripper" parent_link="ee_gripper_link" group="gripper" parent_group="arm"/>
+    <end_effector name="gripper" parent_link="${tf_prefix}ee_gripper_link" group="gripper" parent_group="arm"/>
     <!--DISABLE COLLISIONS: By default it is assumed that any link of the robot could potentially come into collision with any other link in the robot. This tag disables collision checking between a specified pair of links. -->
-    <disable_collisions link1="base_link" link2="link_1" reason="Adjacent"/>
-    <disable_collisions link1="base_link" link2="link_2" reason="Never"/>
-    <disable_collisions link1="carriage_left" link2="carriage_right" reason="Never"/>
-    <disable_collisions link1="carriage_left" link2="gripper_left" reason="Adjacent"/>
-    <disable_collisions link1="carriage_left" link2="gripper_right" reason="Never"/>
-    <disable_collisions link1="carriage_left" link2="link_3" reason="Never"/>
-    <disable_collisions link1="carriage_left" link2="link_4" reason="Never"/>
-    <disable_collisions link1="carriage_left" link2="link_5" reason="Never"/>
-    <disable_collisions link1="carriage_left" link2="link_6" reason="Adjacent"/>
-    <disable_collisions link1="carriage_right" link2="gripper_left" reason="Never"/>
-    <disable_collisions link1="carriage_right" link2="gripper_right" reason="Adjacent"/>
-    <disable_collisions link1="carriage_right" link2="link_3" reason="Never"/>
-    <disable_collisions link1="carriage_right" link2="link_4" reason="Never"/>
-    <disable_collisions link1="carriage_right" link2="link_5" reason="Never"/>
-    <disable_collisions link1="carriage_right" link2="link_6" reason="Adjacent"/>
-    <disable_collisions link1="gripper_left" link2="gripper_right" reason="Never"/>
-    <disable_collisions link1="gripper_left" link2="link_3" reason="Never"/>
-    <disable_collisions link1="gripper_left" link2="link_4" reason="Never"/>
-    <disable_collisions link1="gripper_left" link2="link_5" reason="Never"/>
-    <disable_collisions link1="gripper_left" link2="link_6" reason="Default"/>
-    <disable_collisions link1="gripper_right" link2="link_3" reason="Never"/>
-    <disable_collisions link1="gripper_right" link2="link_4" reason="Never"/>
-    <disable_collisions link1="gripper_right" link2="link_5" reason="Never"/>
-    <disable_collisions link1="gripper_right" link2="link_6" reason="Default"/>
-    <disable_collisions link1="link_1" link2="link_2" reason="Adjacent"/>
-    <disable_collisions link1="link_2" link2="link_3" reason="Adjacent"/>
-    <disable_collisions link1="link_2" link2="link_5" reason="Adjacent"/>  <!-- links 2 and 5 are in contact at rest -->
-    <disable_collisions link1="link_3" link2="link_4" reason="Adjacent"/>
-    <disable_collisions link1="link_3" link2="link_5" reason="Never"/>
-    <disable_collisions link1="link_3" link2="link_6" reason="Never"/>
-    <disable_collisions link1="link_4" link2="link_5" reason="Adjacent"/>
-    <disable_collisions link1="link_4" link2="link_6" reason="Never"/>
-    <disable_collisions link1="link_5" link2="link_6" reason="Adjacent"/>
+    <disable_collisions link1="${tf_prefix}base_link" link2="${tf_prefix}link_1" reason="Adjacent"/>
+    <disable_collisions link1="${tf_prefix}base_link" link2="${tf_prefix}link_2" reason="Never"/>
+    <disable_collisions link1="${tf_prefix}carriage_left" link2="${tf_prefix}carriage_right" reason="Never"/>
+    <disable_collisions link1="${tf_prefix}carriage_left" link2="${tf_prefix}gripper_left" reason="Adjacent"/>
+    <disable_collisions link1="${tf_prefix}carriage_left" link2="${tf_prefix}gripper_right" reason="Never"/>
+    <disable_collisions link1="${tf_prefix}carriage_left" link2="${tf_prefix}link_3" reason="Never"/>
+    <disable_collisions link1="${tf_prefix}carriage_left" link2="${tf_prefix}link_4" reason="Never"/>
+    <disable_collisions link1="${tf_prefix}carriage_left" link2="${tf_prefix}link_5" reason="Never"/>
+    <disable_collisions link1="${tf_prefix}carriage_left" link2="${tf_prefix}link_6" reason="Adjacent"/>
+    <disable_collisions link1="${tf_prefix}carriage_right" link2="${tf_prefix}gripper_left" reason="Never"/>
+    <disable_collisions link1="${tf_prefix}carriage_right" link2="${tf_prefix}gripper_right" reason="Adjacent"/>
+    <disable_collisions link1="${tf_prefix}carriage_right" link2="${tf_prefix}link_3" reason="Never"/>
+    <disable_collisions link1="${tf_prefix}carriage_right" link2="${tf_prefix}link_4" reason="Never"/>
+    <disable_collisions link1="${tf_prefix}carriage_right" link2="${tf_prefix}link_5" reason="Never"/>
+    <disable_collisions link1="${tf_prefix}carriage_right" link2="${tf_prefix}link_6" reason="Adjacent"/>
+    <disable_collisions link1="${tf_prefix}gripper_left" link2="${tf_prefix}gripper_right" reason="Never"/>
+    <disable_collisions link1="${tf_prefix}gripper_left" link2="${tf_prefix}link_3" reason="Never"/>
+    <disable_collisions link1="${tf_prefix}gripper_left" link2="${tf_prefix}link_4" reason="Never"/>
+    <disable_collisions link1="${tf_prefix}gripper_left" link2="${tf_prefix}link_5" reason="Never"/>
+    <disable_collisions link1="${tf_prefix}gripper_left" link2="${tf_prefix}link_6" reason="Default"/>
+    <disable_collisions link1="${tf_prefix}gripper_right" link2="${tf_prefix}link_3" reason="Never"/>
+    <disable_collisions link1="${tf_prefix}gripper_right" link2="${tf_prefix}link_4" reason="Never"/>
+    <disable_collisions link1="${tf_prefix}gripper_right" link2="${tf_prefix}link_5" reason="Never"/>
+    <disable_collisions link1="${tf_prefix}gripper_right" link2="${tf_prefix}link_6" reason="Default"/>
+    <disable_collisions link1="${tf_prefix}link_1" link2="${tf_prefix}link_2" reason="Adjacent"/>
+    <disable_collisions link1="${tf_prefix}link_2" link2="${tf_prefix}link_3" reason="Adjacent"/>
+    <disable_collisions link1="${tf_prefix}link_2" link2="${tf_prefix}link_5" reason="Adjacent"/>  <!-- links 2 and 5 are in contact at rest -->
+    <disable_collisions link1="${tf_prefix}link_3" link2="${tf_prefix}link_4" reason="Adjacent"/>
+    <disable_collisions link1="${tf_prefix}link_3" link2="${tf_prefix}link_5" reason="Never"/>
+    <disable_collisions link1="${tf_prefix}link_3" link2="${tf_prefix}link_6" reason="Never"/>
+    <disable_collisions link1="${tf_prefix}link_4" link2="${tf_prefix}link_5" reason="Adjacent"/>
+    <disable_collisions link1="${tf_prefix}link_4" link2="${tf_prefix}link_6" reason="Never"/>
+    <disable_collisions link1="${tf_prefix}link_5" link2="${tf_prefix}link_6" reason="Adjacent"/>
+    <disable_collisions link1="${tf_prefix}Custom_Mount" link2="${tf_prefix}base_link" reason="Default"/>
+    <disable_collisions link1="${tf_prefix}Custom_Mount" link2="${tf_prefix}link_1" reason="Default"/>
+    <disable_collisions link1="${tf_prefix}Custom_Mount" link2="${tf_prefix}link_2" reason="Default"/>
+    <disable_collisions link1="${tf_prefix}Custom_Mount" link2="${tf_prefix}link_5" reason="Default"/>
+    <disable_collisions link1="${tf_prefix}Custom_Mount" link2="${tf_prefix}link_6" reason="Adjacent"/>
+    <disable_collisions link1="${tf_prefix}Custom_Mount" link2="${tf_prefix}carriage_left" reason="Never"/>
+    <disable_collisions link1="${tf_prefix}Custom_Mount" link2="${tf_prefix}carriage_right" reason="Never"/>
+    <disable_collisions link1="${tf_prefix}Custom_Mount" link2="${tf_prefix}gripper_left" reason="Never"/>
+    <disable_collisions link1="${tf_prefix}Custom_Mount" link2="${tf_prefix}gripper_right" reason="Never"/>
+    <disable_collisions link1="${tf_prefix}Top_Camera_frame" link2="${tf_prefix}base_link" reason="Never"/>
+    <disable_collisions link1="${tf_prefix}Top_Camera_frame" link2="${tf_prefix}link_1" reason="Never"/>
+    <disable_collisions link1="${tf_prefix}Top_Camera_frame" link2="${tf_prefix}link_2" reason="Never"/>
+    <!--DISABLE COLLISIONS: By default it is assumed that any link of the robot could potentially come into collision with any other link in the robot. This tag disables collision checking between a specified pair of links. -->
+    <xacro:if value="${srdf_use_downdraft}">
+        <disable_collisions link1="${tf_prefix}Back_Plate_Exhaust" link2="${tf_prefix}Bottom_Box" reason="Never"/>
+        <disable_collisions link1="${tf_prefix}Back_Plate_Exhaust" link2="${tf_prefix}Chute_01" reason="Never"/>
+        <disable_collisions link1="${tf_prefix}Back_Plate_Exhaust" link2="${tf_prefix}Chute_02" reason="Never"/>
+        <disable_collisions link1="${tf_prefix}Back_Plate_Exhaust" link2="${tf_prefix}Chute_03" reason="Never"/>
+        <disable_collisions link1="${tf_prefix}Back_Plate_Exhaust" link2="${tf_prefix}Custom_Mount" reason="Never"/>
+        <disable_collisions link1="${tf_prefix}Back_Plate_Exhaust" link2="${tf_prefix}Top_Camera_frame" reason="Never"/>
+        <disable_collisions link1="${tf_prefix}Custom_Mount" link2="${tf_prefix}Side_Plates_Right" reason="Never"/>
+        <disable_collisions link1="${tf_prefix}Custom_Mount" link2="${tf_prefix}base_mount" reason="Never"/>
+        <disable_collisions link1="${tf_prefix}Custom_Mount" link2="${tf_prefix}light_1" reason="Never"/>
+        <disable_collisions link1="${tf_prefix}Custom_Mount" link2="${tf_prefix}pillar_1" reason="Never"/>
+        <disable_collisions link1="${tf_prefix}Custom_Mount" link2="${tf_prefix}pillar_2" reason="Never"/>
+        <disable_collisions link1="${tf_prefix}Custom_Mount" link2="${tf_prefix}pillar_3" reason="Never"/>
+        <disable_collisions link1="${tf_prefix}Custom_Mount" link2="${tf_prefix}pillar_4" reason="Never"/>
+        <disable_collisions link1="${tf_prefix}Custom_Mount" link2="${tf_prefix}suction_cup" reason="Never"/>
+        <disable_collisions link1="${tf_prefix}Custom_Mount" link2="${tf_prefix}suction_mount" reason="Never"/>
+        <disable_collisions link1="${tf_prefix}Custom_Mount" link2="${tf_prefix}tube" reason="Never"/>
+        <disable_collisions link1="${tf_prefix}Back_Plate_Exhaust" link2="${tf_prefix}Front_Weld_Plate" reason="Never"/>
+        <disable_collisions link1="${tf_prefix}Back_Plate_Exhaust" link2="${tf_prefix}Letter_Trimmer_Holder" reason="Never"/>
+        <disable_collisions link1="${tf_prefix}Back_Plate_Exhaust" link2="${tf_prefix}Mail_Spreader_Housing" reason="Never"/>
+        <disable_collisions link1="${tf_prefix}Back_Plate_Exhaust" link2="${tf_prefix}Mail_Top_Plate" reason="Never"/>
+        <disable_collisions link1="${tf_prefix}Back_Plate_Exhaust" link2="${tf_prefix}Pedestal" reason="Never"/>
+        <disable_collisions link1="${tf_prefix}Back_Plate_Exhaust" link2="${tf_prefix}RealSense_D405" reason="Never"/>
+        <disable_collisions link1="${tf_prefix}Back_Plate_Exhaust" link2="${tf_prefix}RealSense_Holder_01" reason="Never"/>
+        <disable_collisions link1="${tf_prefix}Back_Plate_Exhaust" link2="${tf_prefix}RealSense_Holder_02" reason="Never"/>
+        <disable_collisions link1="${tf_prefix}Back_Plate_Exhaust" link2="${tf_prefix}Rear_Panel" reason="Never"/>
+        <disable_collisions link1="${tf_prefix}Back_Plate_Exhaust" link2="${tf_prefix}Side_Plates_Left" reason="Default"/>
+        <disable_collisions link1="${tf_prefix}Back_Plate_Exhaust" link2="${tf_prefix}Side_Plates_Right" reason="Never"/>
+        <disable_collisions link1="${tf_prefix}Back_Plate_Exhaust" link2="${tf_prefix}Top_Panel" reason="Adjacent"/>
+        <disable_collisions link1="${tf_prefix}Back_Plate_Exhaust" link2="${tf_prefix}Top_Weld_Plate" reason="Default"/>
+        <disable_collisions link1="${tf_prefix}Back_Plate_Exhaust" link2="${tf_prefix}Vibration_Table_Plate" reason="Never"/>
+        <disable_collisions link1="${tf_prefix}Back_Plate_Exhaust" link2="${tf_prefix}Vibration_Table_Top_Plate" reason="Never"/>
+        <disable_collisions link1="${tf_prefix}Back_Plate_Exhaust" link2="${tf_prefix}base_link" reason="Never"/>
+        <disable_collisions link1="${tf_prefix}Back_Plate_Exhaust" link2="${tf_prefix}base_mount" reason="Never"/>
+        <disable_collisions link1="${tf_prefix}Back_Plate_Exhaust" link2="${tf_prefix}carriage_left" reason="Never"/>
+        <disable_collisions link1="${tf_prefix}Back_Plate_Exhaust" link2="${tf_prefix}carriage_right" reason="Never"/>
+        <disable_collisions link1="${tf_prefix}Back_Plate_Exhaust" link2="${tf_prefix}gripper_left" reason="Never"/>
+        <disable_collisions link1="${tf_prefix}Back_Plate_Exhaust" link2="${tf_prefix}gripper_right" reason="Never"/>
+        <disable_collisions link1="${tf_prefix}Back_Plate_Exhaust" link2="${tf_prefix}light_1" reason="Never"/>
+        <disable_collisions link1="${tf_prefix}Back_Plate_Exhaust" link2="${tf_prefix}light_2" reason="Never"/>
+        <disable_collisions link1="${tf_prefix}Back_Plate_Exhaust" link2="${tf_prefix}link_1" reason="Never"/>
+        <disable_collisions link1="${tf_prefix}Back_Plate_Exhaust" link2="${tf_prefix}link_2" reason="Never"/>
+        <disable_collisions link1="${tf_prefix}Back_Plate_Exhaust" link2="${tf_prefix}link_3" reason="Never"/>
+        <disable_collisions link1="${tf_prefix}Back_Plate_Exhaust" link2="${tf_prefix}link_4" reason="Never"/>
+        <disable_collisions link1="${tf_prefix}Back_Plate_Exhaust" link2="${tf_prefix}link_5" reason="Never"/>
+        <disable_collisions link1="${tf_prefix}Back_Plate_Exhaust" link2="${tf_prefix}link_6" reason="Never"/>
+        <disable_collisions link1="${tf_prefix}Back_Plate_Exhaust" link2="${tf_prefix}pillar_1" reason="Never"/>
+        <disable_collisions link1="${tf_prefix}Back_Plate_Exhaust" link2="${tf_prefix}pillar_2" reason="Never"/>
+        <disable_collisions link1="${tf_prefix}Back_Plate_Exhaust" link2="${tf_prefix}pillar_3" reason="Never"/>
+        <disable_collisions link1="${tf_prefix}Back_Plate_Exhaust" link2="${tf_prefix}pillar_4" reason="Never"/>
+        <disable_collisions link1="${tf_prefix}Back_Plate_Exhaust" link2="${tf_prefix}suction_cup" reason="Never"/>
+        <disable_collisions link1="${tf_prefix}Back_Plate_Exhaust" link2="${tf_prefix}suction_mount" reason="Never"/>
+        <disable_collisions link1="${tf_prefix}Back_Plate_Exhaust" link2="${tf_prefix}tube" reason="Never"/>
+        <disable_collisions link1="${tf_prefix}Bottom_Box" link2="${tf_prefix}Chute_01" reason="Never"/>
+        <disable_collisions link1="${tf_prefix}Bottom_Box" link2="${tf_prefix}Chute_02" reason="Never"/>
+        <disable_collisions link1="${tf_prefix}Bottom_Box" link2="${tf_prefix}Chute_03" reason="Never"/>
+        <disable_collisions link1="${tf_prefix}Bottom_Box" link2="${tf_prefix}Front_Weld_Plate" reason="Never"/>
+        <disable_collisions link1="${tf_prefix}Bottom_Box" link2="${tf_prefix}Letter_Trimmer_Holder" reason="Never"/>
+        <disable_collisions link1="${tf_prefix}Bottom_Box" link2="${tf_prefix}Mail_Spreader_Housing" reason="Never"/>
+        <disable_collisions link1="${tf_prefix}Bottom_Box" link2="${tf_prefix}Mail_Top_Plate" reason="Never"/>
+        <disable_collisions link1="${tf_prefix}Bottom_Box" link2="${tf_prefix}Pedestal" reason="Adjacent"/>
+        <disable_collisions link1="${tf_prefix}Bottom_Box" link2="${tf_prefix}RealSense_D405" reason="Never"/>
+        <disable_collisions link1="${tf_prefix}Bottom_Box" link2="${tf_prefix}RealSense_Holder_01" reason="Never"/>
+        <disable_collisions link1="${tf_prefix}Bottom_Box" link2="${tf_prefix}RealSense_Holder_02" reason="Never"/>
+        <disable_collisions link1="${tf_prefix}Bottom_Box" link2="${tf_prefix}Rear_Panel" reason="Never"/>
+        <disable_collisions link1="${tf_prefix}Bottom_Box" link2="${tf_prefix}Side_Plates_Left" reason="Never"/>
+        <disable_collisions link1="${tf_prefix}Bottom_Box" link2="${tf_prefix}Side_Plates_Right" reason="Never"/>
+        <disable_collisions link1="${tf_prefix}Bottom_Box" link2="${tf_prefix}Top_Panel" reason="Adjacent"/>
+        <disable_collisions link1="${tf_prefix}Bottom_Box" link2="${tf_prefix}Top_Weld_Plate" reason="Never"/>
+        <disable_collisions link1="${tf_prefix}Bottom_Box" link2="${tf_prefix}Vibration_Table_Plate" reason="Never"/>
+        <disable_collisions link1="${tf_prefix}Bottom_Box" link2="${tf_prefix}Vibration_Table_Top_Plate" reason="Never"/>
+        <disable_collisions link1="${tf_prefix}Bottom_Box" link2="${tf_prefix}base_link" reason="Adjacent"/>
+        <disable_collisions link1="${tf_prefix}Bottom_Box" link2="${tf_prefix}light_1" reason="Never"/>
+        <disable_collisions link1="${tf_prefix}Bottom_Box" link2="${tf_prefix}light_2" reason="Never"/>
+        <disable_collisions link1="${tf_prefix}Bottom_Box" link2="${tf_prefix}link_1" reason="Never"/>
+        <disable_collisions link1="${tf_prefix}Bottom_Box" link2="${tf_prefix}link_2" reason="Never"/>
+        <disable_collisions link1="${tf_prefix}Bottom_Box" link2="${tf_prefix}Top_Camera_frame" reason="Adjacent"/>
+        <disable_collisions link1="${tf_prefix}Chute_01" link2="${tf_prefix}Chute_02" reason="Adjacent"/>
+        <disable_collisions link1="${tf_prefix}Chute_01" link2="${tf_prefix}Chute_03" reason="Adjacent"/>
+        <disable_collisions link1="${tf_prefix}Chute_01" link2="${tf_prefix}Front_Weld_Plate" reason="Default"/>
+        <disable_collisions link1="${tf_prefix}Chute_01" link2="${tf_prefix}Letter_Trimmer_Holder" reason="Never"/>
+        <disable_collisions link1="${tf_prefix}Chute_01" link2="${tf_prefix}Mail_Spreader_Housing" reason="Default"/>
+        <disable_collisions link1="${tf_prefix}Chute_01" link2="${tf_prefix}Mail_Top_Plate" reason="Never"/>
+        <disable_collisions link1="${tf_prefix}Chute_01" link2="${tf_prefix}Pedestal" reason="Never"/>
+        <disable_collisions link1="${tf_prefix}Chute_01" link2="${tf_prefix}RealSense_D405" reason="Never"/>
+        <disable_collisions link1="${tf_prefix}Chute_01" link2="${tf_prefix}RealSense_Holder_01" reason="Never"/>
+        <disable_collisions link1="${tf_prefix}Chute_01" link2="${tf_prefix}RealSense_Holder_02" reason="Never"/>
+        <disable_collisions link1="${tf_prefix}Chute_01" link2="${tf_prefix}Rear_Panel" reason="Never"/>
+        <disable_collisions link1="${tf_prefix}Chute_01" link2="${tf_prefix}Side_Plates_Left" reason="Never"/>
+        <disable_collisions link1="${tf_prefix}Chute_01" link2="${tf_prefix}Side_Plates_Right" reason="Never"/>
+        <disable_collisions link1="${tf_prefix}Chute_01" link2="${tf_prefix}Top_Panel" reason="Adjacent"/>
+        <disable_collisions link1="${tf_prefix}Chute_01" link2="${tf_prefix}Top_Weld_Plate" reason="Never"/>
+        <disable_collisions link1="${tf_prefix}Chute_01" link2="${tf_prefix}Vibration_Table_Plate" reason="Never"/>
+        <disable_collisions link1="${tf_prefix}Chute_01" link2="${tf_prefix}Vibration_Table_Top_Plate" reason="Never"/>
+        <disable_collisions link1="${tf_prefix}Chute_01" link2="${tf_prefix}base_link" reason="Never"/>
+        <disable_collisions link1="${tf_prefix}Chute_01" link2="${tf_prefix}light_1" reason="Never"/>
+        <disable_collisions link1="${tf_prefix}Chute_01" link2="${tf_prefix}light_2" reason="Never"/>
+        <disable_collisions link1="${tf_prefix}Chute_01" link2="${tf_prefix}link_1" reason="Never"/>
+        <disable_collisions link1="${tf_prefix}Chute_01" link2="${tf_prefix}link_2" reason="Never"/>
+        <disable_collisions link1="${tf_prefix}Chute_01" link2="${tf_prefix}Top_Camera_frame" reason="Never"/>
+        <disable_collisions link1="${tf_prefix}Chute_02" link2="${tf_prefix}Chute_03" reason="Never"/>
+        <disable_collisions link1="${tf_prefix}Chute_02" link2="${tf_prefix}Front_Weld_Plate" reason="Never"/>
+        <disable_collisions link1="${tf_prefix}Chute_02" link2="${tf_prefix}Letter_Trimmer_Holder" reason="Never"/>
+        <disable_collisions link1="${tf_prefix}Chute_02" link2="${tf_prefix}Mail_Spreader_Housing" reason="Default"/>
+        <disable_collisions link1="${tf_prefix}Chute_02" link2="${tf_prefix}Mail_Top_Plate" reason="Never"/>
+        <disable_collisions link1="${tf_prefix}Chute_02" link2="${tf_prefix}Pedestal" reason="Never"/>
+        <disable_collisions link1="${tf_prefix}Chute_02" link2="${tf_prefix}RealSense_D405" reason="Never"/>
+        <disable_collisions link1="${tf_prefix}Chute_02" link2="${tf_prefix}RealSense_Holder_01" reason="Never"/>
+        <disable_collisions link1="${tf_prefix}Chute_02" link2="${tf_prefix}RealSense_Holder_02" reason="Never"/>
+        <disable_collisions link1="${tf_prefix}Chute_02" link2="${tf_prefix}Rear_Panel" reason="Never"/>
+        <disable_collisions link1="${tf_prefix}Chute_02" link2="${tf_prefix}Side_Plates_Left" reason="Never"/>
+        <disable_collisions link1="${tf_prefix}Chute_02" link2="${tf_prefix}Side_Plates_Right" reason="Never"/>
+        <disable_collisions link1="${tf_prefix}Chute_02" link2="${tf_prefix}Top_Panel" reason="Never"/>
+        <disable_collisions link1="${tf_prefix}Chute_02" link2="${tf_prefix}Top_Weld_Plate" reason="Never"/>
+        <disable_collisions link1="${tf_prefix}Chute_02" link2="${tf_prefix}Vibration_Table_Plate" reason="Never"/>
+        <disable_collisions link1="${tf_prefix}Chute_02" link2="${tf_prefix}Vibration_Table_Top_Plate" reason="Never"/>
+        <disable_collisions link1="${tf_prefix}Chute_02" link2="${tf_prefix}base_link" reason="Never"/>
+        <disable_collisions link1="${tf_prefix}Chute_02" link2="${tf_prefix}light_1" reason="Never"/>
+        <disable_collisions link1="${tf_prefix}Chute_02" link2="${tf_prefix}light_2" reason="Never"/>
+        <disable_collisions link1="${tf_prefix}Chute_02" link2="${tf_prefix}link_1" reason="Never"/>
+        <disable_collisions link1="${tf_prefix}Chute_02" link2="${tf_prefix}Top_Camera_frame" reason="Never"/>
+        <disable_collisions link1="${tf_prefix}Chute_03" link2="${tf_prefix}Front_Weld_Plate" reason="Default"/>
+        <disable_collisions link1="${tf_prefix}Chute_03" link2="${tf_prefix}Letter_Trimmer_Holder" reason="Never"/>
+        <disable_collisions link1="${tf_prefix}Chute_03" link2="${tf_prefix}Mail_Spreader_Housing" reason="Never"/>
+        <disable_collisions link1="${tf_prefix}Chute_03" link2="${tf_prefix}Mail_Top_Plate" reason="Never"/>
+        <disable_collisions link1="${tf_prefix}Chute_03" link2="${tf_prefix}Pedestal" reason="Never"/>
+        <disable_collisions link1="${tf_prefix}Chute_03" link2="${tf_prefix}RealSense_D405" reason="Never"/>
+        <disable_collisions link1="${tf_prefix}Chute_03" link2="${tf_prefix}RealSense_Holder_01" reason="Never"/>
+        <disable_collisions link1="${tf_prefix}Chute_03" link2="${tf_prefix}RealSense_Holder_02" reason="Never"/>
+        <disable_collisions link1="${tf_prefix}Chute_03" link2="${tf_prefix}Rear_Panel" reason="Never"/>
+        <disable_collisions link1="${tf_prefix}Chute_03" link2="${tf_prefix}Side_Plates_Left" reason="Never"/>
+        <disable_collisions link1="${tf_prefix}Chute_03" link2="${tf_prefix}Side_Plates_Right" reason="Never"/>
+        <disable_collisions link1="${tf_prefix}Chute_03" link2="${tf_prefix}Top_Panel" reason="Never"/>
+        <disable_collisions link1="${tf_prefix}Chute_03" link2="${tf_prefix}Top_Weld_Plate" reason="Never"/>
+        <disable_collisions link1="${tf_prefix}Chute_03" link2="${tf_prefix}Vibration_Table_Plate" reason="Never"/>
+        <disable_collisions link1="${tf_prefix}Chute_03" link2="${tf_prefix}Vibration_Table_Top_Plate" reason="Never"/>
+        <disable_collisions link1="${tf_prefix}Chute_03" link2="${tf_prefix}base_link" reason="Never"/>
+        <disable_collisions link1="${tf_prefix}Chute_03" link2="${tf_prefix}light_1" reason="Never"/>
+        <disable_collisions link1="${tf_prefix}Chute_03" link2="${tf_prefix}light_2" reason="Never"/>
+        <disable_collisions link1="${tf_prefix}Chute_03" link2="${tf_prefix}link_1" reason="Never"/>
+        <disable_collisions link1="${tf_prefix}Chute_03" link2="${tf_prefix}link_2" reason="Never"/>
+        <disable_collisions link1="${tf_prefix}Chute_03" link2="${tf_prefix}Top_Camera_frame" reason="Never"/>
+        <disable_collisions link1="${tf_prefix}Front_Weld_Plate" link2="${tf_prefix}Letter_Trimmer_Holder" reason="Never"/>
+        <disable_collisions link1="${tf_prefix}Front_Weld_Plate" link2="${tf_prefix}Mail_Spreader_Housing" reason="Never"/>
+        <disable_collisions link1="${tf_prefix}Front_Weld_Plate" link2="${tf_prefix}Mail_Top_Plate" reason="Never"/>
+        <disable_collisions link1="${tf_prefix}Front_Weld_Plate" link2="${tf_prefix}Pedestal" reason="Never"/>
+        <disable_collisions link1="${tf_prefix}Front_Weld_Plate" link2="${tf_prefix}RealSense_D405" reason="Never"/>
+        <disable_collisions link1="${tf_prefix}Front_Weld_Plate" link2="${tf_prefix}RealSense_Holder_01" reason="Never"/>
+        <disable_collisions link1="${tf_prefix}Front_Weld_Plate" link2="${tf_prefix}RealSense_Holder_02" reason="Never"/>
+        <disable_collisions link1="${tf_prefix}Front_Weld_Plate" link2="${tf_prefix}Rear_Panel" reason="Never"/>
+        <disable_collisions link1="${tf_prefix}Front_Weld_Plate" link2="${tf_prefix}Side_Plates_Left" reason="Default"/>
+        <disable_collisions link1="${tf_prefix}Front_Weld_Plate" link2="${tf_prefix}Side_Plates_Right" reason="Never"/>
+        <disable_collisions link1="${tf_prefix}Front_Weld_Plate" link2="${tf_prefix}Top_Panel" reason="Adjacent"/>
+        <disable_collisions link1="${tf_prefix}Front_Weld_Plate" link2="${tf_prefix}Top_Weld_Plate" reason="Never"/>
+        <disable_collisions link1="${tf_prefix}Front_Weld_Plate" link2="${tf_prefix}Vibration_Table_Plate" reason="Never"/>
+        <disable_collisions link1="${tf_prefix}Front_Weld_Plate" link2="${tf_prefix}Vibration_Table_Top_Plate" reason="Never"/>
+        <disable_collisions link1="${tf_prefix}Front_Weld_Plate" link2="${tf_prefix}base_link" reason="Never"/>
+        <disable_collisions link1="${tf_prefix}Front_Weld_Plate" link2="${tf_prefix}light_1" reason="Never"/>
+        <disable_collisions link1="${tf_prefix}Front_Weld_Plate" link2="${tf_prefix}light_2" reason="Never"/>
+        <disable_collisions link1="${tf_prefix}Front_Weld_Plate" link2="${tf_prefix}link_1" reason="Never"/>
+        <disable_collisions link1="${tf_prefix}Front_Weld_Plate" link2="${tf_prefix}Top_Camera_frame" reason="Never"/>
+        <disable_collisions link1="${tf_prefix}Letter_Trimmer_Holder" link2="${tf_prefix}Mail_Spreader_Housing" reason="Adjacent"/>
+        <disable_collisions link1="${tf_prefix}Letter_Trimmer_Holder" link2="${tf_prefix}Mail_Top_Plate" reason="Never"/>
+        <disable_collisions link1="${tf_prefix}Letter_Trimmer_Holder" link2="${tf_prefix}Pedestal" reason="Never"/>
+        <disable_collisions link1="${tf_prefix}Letter_Trimmer_Holder" link2="${tf_prefix}RealSense_D405" reason="Never"/>
+        <disable_collisions link1="${tf_prefix}Letter_Trimmer_Holder" link2="${tf_prefix}RealSense_Holder_01" reason="Never"/>
+        <disable_collisions link1="${tf_prefix}Letter_Trimmer_Holder" link2="${tf_prefix}RealSense_Holder_02" reason="Never"/>
+        <disable_collisions link1="${tf_prefix}Letter_Trimmer_Holder" link2="${tf_prefix}Rear_Panel" reason="Never"/>
+        <disable_collisions link1="${tf_prefix}Letter_Trimmer_Holder" link2="${tf_prefix}Side_Plates_Left" reason="Never"/>
+        <disable_collisions link1="${tf_prefix}Letter_Trimmer_Holder" link2="${tf_prefix}Side_Plates_Right" reason="Never"/>
+        <disable_collisions link1="${tf_prefix}Letter_Trimmer_Holder" link2="${tf_prefix}Top_Panel" reason="Never"/>
+        <disable_collisions link1="${tf_prefix}Letter_Trimmer_Holder" link2="${tf_prefix}Top_Weld_Plate" reason="Never"/>
+        <disable_collisions link1="${tf_prefix}Letter_Trimmer_Holder" link2="${tf_prefix}Vibration_Table_Plate" reason="Never"/>
+        <disable_collisions link1="${tf_prefix}Letter_Trimmer_Holder" link2="${tf_prefix}Vibration_Table_Top_Plate" reason="Never"/>
+        <disable_collisions link1="${tf_prefix}Letter_Trimmer_Holder" link2="${tf_prefix}base_link" reason="Never"/>
+        <disable_collisions link1="${tf_prefix}Letter_Trimmer_Holder" link2="${tf_prefix}light_1" reason="Never"/>
+        <disable_collisions link1="${tf_prefix}Letter_Trimmer_Holder" link2="${tf_prefix}light_2" reason="Never"/>
+        <disable_collisions link1="${tf_prefix}Letter_Trimmer_Holder" link2="${tf_prefix}link_1" reason="Never"/>
+        <disable_collisions link1="${tf_prefix}Letter_Trimmer_Holder" link2="${tf_prefix}Top_Camera_frame" reason="Never"/>
+        <disable_collisions link1="${tf_prefix}Mail_Spreader_Housing" link2="${tf_prefix}Mail_Top_Plate" reason="Adjacent"/>
+        <disable_collisions link1="${tf_prefix}Mail_Spreader_Housing" link2="${tf_prefix}Pedestal" reason="Never"/>
+        <disable_collisions link1="${tf_prefix}Mail_Spreader_Housing" link2="${tf_prefix}RealSense_D405" reason="Never"/>
+        <disable_collisions link1="${tf_prefix}Mail_Spreader_Housing" link2="${tf_prefix}RealSense_Holder_01" reason="Never"/>
+        <disable_collisions link1="${tf_prefix}Mail_Spreader_Housing" link2="${tf_prefix}RealSense_Holder_02" reason="Never"/>
+        <disable_collisions link1="${tf_prefix}Mail_Spreader_Housing" link2="${tf_prefix}Rear_Panel" reason="Never"/>
+        <disable_collisions link1="${tf_prefix}Mail_Spreader_Housing" link2="${tf_prefix}Side_Plates_Left" reason="Never"/>
+        <disable_collisions link1="${tf_prefix}Mail_Spreader_Housing" link2="${tf_prefix}Side_Plates_Right" reason="Never"/>
+        <disable_collisions link1="${tf_prefix}Mail_Spreader_Housing" link2="${tf_prefix}Top_Panel" reason="Adjacent"/>
+        <disable_collisions link1="${tf_prefix}Mail_Spreader_Housing" link2="${tf_prefix}Top_Weld_Plate" reason="Never"/>
+        <disable_collisions link1="${tf_prefix}Mail_Spreader_Housing" link2="${tf_prefix}Vibration_Table_Plate" reason="Never"/>
+        <disable_collisions link1="${tf_prefix}Mail_Spreader_Housing" link2="${tf_prefix}Vibration_Table_Top_Plate" reason="Never"/>
+        <disable_collisions link1="${tf_prefix}Mail_Spreader_Housing" link2="${tf_prefix}base_link" reason="Never"/>
+        <disable_collisions link1="${tf_prefix}Mail_Spreader_Housing" link2="${tf_prefix}carriage_left" reason="Default"/>
+        <disable_collisions link1="${tf_prefix}Mail_Spreader_Housing" link2="${tf_prefix}carriage_right" reason="Default"/>
+        <disable_collisions link1="${tf_prefix}Mail_Spreader_Housing" link2="${tf_prefix}gripper_left" reason="Default"/>
+        <disable_collisions link1="${tf_prefix}Mail_Spreader_Housing" link2="${tf_prefix}gripper_right" reason="Default"/>
+        <disable_collisions link1="${tf_prefix}Mail_Spreader_Housing" link2="${tf_prefix}light_1" reason="Never"/>
+        <disable_collisions link1="${tf_prefix}Mail_Spreader_Housing" link2="${tf_prefix}light_2" reason="Never"/>
+        <disable_collisions link1="${tf_prefix}Mail_Spreader_Housing" link2="${tf_prefix}link_1" reason="Never"/>
+        <disable_collisions link1="${tf_prefix}Mail_Spreader_Housing" link2="${tf_prefix}link_6" reason="Default"/>
+        <disable_collisions link1="${tf_prefix}Mail_Spreader_Housing" link2="${tf_prefix}Top_Camera_frame" reason="Never"/>
+        <disable_collisions link1="${tf_prefix}Mail_Top_Plate" link2="${tf_prefix}Pedestal" reason="Never"/>
+        <disable_collisions link1="${tf_prefix}Mail_Top_Plate" link2="${tf_prefix}RealSense_D405" reason="Never"/>
+        <disable_collisions link1="${tf_prefix}Mail_Top_Plate" link2="${tf_prefix}RealSense_Holder_01" reason="Never"/>
+        <disable_collisions link1="${tf_prefix}Mail_Top_Plate" link2="${tf_prefix}RealSense_Holder_02" reason="Never"/>
+        <disable_collisions link1="${tf_prefix}Mail_Top_Plate" link2="${tf_prefix}Rear_Panel" reason="Never"/>
+        <disable_collisions link1="${tf_prefix}Mail_Top_Plate" link2="${tf_prefix}Side_Plates_Left" reason="Never"/>
+        <disable_collisions link1="${tf_prefix}Mail_Top_Plate" link2="${tf_prefix}Side_Plates_Right" reason="Never"/>
+        <disable_collisions link1="${tf_prefix}Mail_Top_Plate" link2="${tf_prefix}Top_Panel" reason="Never"/>
+        <disable_collisions link1="${tf_prefix}Mail_Top_Plate" link2="${tf_prefix}Top_Weld_Plate" reason="Never"/>
+        <disable_collisions link1="${tf_prefix}Mail_Top_Plate" link2="${tf_prefix}Vibration_Table_Plate" reason="Never"/>
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