Commit message: edited srdf

File: trossen_arm_moveit/config/wxai.srdf.xacro (robot description, xacro)
@@ -6,5 +6,7 @@
 <robot name="wxai" xmlns:xacro="http://ros.org/wiki/xacro">
     <xacro:arg name="use_downdraft" default="true"/>
+    <xacro:arg name="use_suction_cup" default="true"/>
     <xacro:property name="srdf_use_downdraft" value="$(arg use_downdraft)"/>
+    <xacro:property name="srdf_use_suction_cup" value="$(arg use_suction_cup)"/>
     <xacro:arg name="prefix" default=""/>
     <xacro:property name="tf_prefix" value="$(arg prefix)"/>
@@ -32,5 +34,5 @@
     </group>
     <group name="gripper">
-        <xacro:if value="${srdf_use_downdraft}">
+        <xacro:if value="${srdf_use_suction_cup}">
             <joint name="${tf_prefix}base_and_suction"/>
             <joint name="${tf_prefix}pillar_1_and_base_mount"/>
@@ -130,4 +132,147 @@
     <disable_collisions link1="${tf_prefix}Top_Camera_frame" link2="${tf_prefix}link_2" reason="Never"/>
     <!--DISABLE COLLISIONS: By default it is assumed that any link of the robot could potentially come into collision with any other link in the robot. This tag disables collision checking between a specified pair of links. -->
+    <xacro:if value="${srdf_use_suction_cup and srdf_use_downdraft}">
+        <disable_collisions link1="${tf_prefix}Back_Plate_Exhaust" link2="${tf_prefix}pillar_1" reason="Never"/>
+        <disable_collisions link1="${tf_prefix}Back_Plate_Exhaust" link2="${tf_prefix}pillar_2" reason="Never"/>
+        <disable_collisions link1="${tf_prefix}Back_Plate_Exhaust" link2="${tf_prefix}pillar_3" reason="Never"/>
+        <disable_collisions link1="${tf_prefix}Back_Plate_Exhaust" link2="${tf_prefix}pillar_4" reason="Never"/>
+        <disable_collisions link1="${tf_prefix}Back_Plate_Exhaust" link2="${tf_prefix}suction_cup" reason="Never"/>
+        <disable_collisions link1="${tf_prefix}Back_Plate_Exhaust" link2="${tf_prefix}suction_mount" reason="Never"/>
+        <disable_collisions link1="${tf_prefix}Back_Plate_Exhaust" link2="${tf_prefix}tube" reason="Never"/>
+        <disable_collisions link1="${tf_prefix}light_1" link2="${tf_prefix}pillar_1" reason="Never"/>
+        <disable_collisions link1="${tf_prefix}light_1" link2="${tf_prefix}pillar_2" reason="Never"/>
+        <disable_collisions link1="${tf_prefix}light_1" link2="${tf_prefix}pillar_3" reason="Never"/>
+        <disable_collisions link1="${tf_prefix}light_1" link2="${tf_prefix}pillar_4" reason="Never"/>
+        <disable_collisions link1="${tf_prefix}light_1" link2="${tf_prefix}suction_cup" reason="Never"/>
+        <disable_collisions link1="${tf_prefix}light_1" link2="${tf_prefix}suction_mount" reason="Never"/>
+        <disable_collisions link1="${tf_prefix}light_1" link2="${tf_prefix}tube" reason="Never"/>
+        <disable_collisions link1="${tf_prefix}light_2" link2="${tf_prefix}link_1" reason="Never"/>
+        <disable_collisions link1="${tf_prefix}light_2" link2="${tf_prefix}link_2" reason="Never"/>
+        <disable_collisions link1="${tf_prefix}light_2" link2="${tf_prefix}link_3" reason="Never"/>
+        <disable_collisions link1="${tf_prefix}light_2" link2="${tf_prefix}link_4" reason="Never"/>
+        <disable_collisions link1="${tf_prefix}light_2" link2="${tf_prefix}link_5" reason="Never"/>
+        <disable_collisions link1="${tf_prefix}light_2" link2="${tf_prefix}pillar_1" reason="Never"/>
+        <disable_collisions link1="${tf_prefix}light_2" link2="${tf_prefix}pillar_2" reason="Never"/>
+        <disable_collisions link1="${tf_prefix}light_2" link2="${tf_prefix}pillar_3" reason="Never"/>
+        <disable_collisions link1="${tf_prefix}light_2" link2="${tf_prefix}pillar_4" reason="Never"/>
+        <disable_collisions link1="${tf_prefix}light_2" link2="${tf_prefix}suction_mount" reason="Never"/>
+        <disable_collisions link1="${tf_prefix}light_2" link2="${tf_prefix}tube" reason="Never"/>
+        <disable_collisions link1="${tf_prefix}Side_Plates_Right" link2="${tf_prefix}pillar_1" reason="Never"/>
+        <disable_collisions link1="${tf_prefix}Side_Plates_Right" link2="${tf_prefix}pillar_2" reason="Never"/>
+        <disable_collisions link1="${tf_prefix}Side_Plates_Right" link2="${tf_prefix}pillar_3" reason="Never"/>
+        <disable_collisions link1="${tf_prefix}Side_Plates_Right" link2="${tf_prefix}pillar_4" reason="Never"/>
+        <disable_collisions link1="${tf_prefix}Side_Plates_Right" link2="${tf_prefix}suction_cup" reason="Never"/>
+        <disable_collisions link1="${tf_prefix}Side_Plates_Right" link2="${tf_prefix}suction_mount" reason="Never"/>
+        <disable_collisions link1="${tf_prefix}Side_Plates_Right" link2="${tf_prefix}tube" reason="Never"/>
+        <disable_collisions link1="${tf_prefix}Top_Weld_Plate" link2="${tf_prefix}pillar_1" reason="Never"/>
+        <disable_collisions link1="${tf_prefix}Top_Weld_Plate" link2="${tf_prefix}pillar_2" reason="Never"/>
+        <disable_collisions link1="${tf_prefix}Top_Weld_Plate" link2="${tf_prefix}pillar_4" reason="Never"/>
+        <disable_collisions link1="${tf_prefix}Top_Weld_Plate" link2="${tf_prefix}suction_mount" reason="Never"/>
+        <disable_collisions link1="${tf_prefix}Top_Weld_Plate" link2="${tf_prefix}tube" reason="Never"/>
+        <disable_collisions link1="${tf_prefix}Rear_Panel" link2="${tf_prefix}pillar_1" reason="Never"/>
+        <disable_collisions link1="${tf_prefix}Rear_Panel" link2="${tf_prefix}pillar_2" reason="Never"/>
+        <disable_collisions link1="${tf_prefix}Rear_Panel" link2="${tf_prefix}pillar_3" reason="Never"/>
+        <disable_collisions link1="${tf_prefix}Rear_Panel" link2="${tf_prefix}pillar_4" reason="Never"/>
+        <disable_collisions link1="${tf_prefix}Rear_Panel" link2="${tf_prefix}tube" reason="Never"/>
+        <disable_collisions link1="${tf_prefix}RealSense_Holder_02" link2="${tf_prefix}pillar_1" reason="Never"/>
+        <disable_collisions link1="${tf_prefix}RealSense_Holder_02" link2="${tf_prefix}pillar_3" reason="Never"/>
+        <disable_collisions link1="${tf_prefix}RealSense_Holder_02" link2="${tf_prefix}tube" reason="Never"/>
+    </xacro:if>
+    <xacro:if value="${srdf_use_suction_cup}">
+        <disable_collisions link1="${tf_prefix}RealSense_D405" link2="${tf_prefix}tube" reason="Never"/>
+        <disable_collisions link1="${tf_prefix}RealSense_D405" link2="${tf_prefix}pillar_1" reason="Never"/>
+        <disable_collisions link1="${tf_prefix}RealSense_D405" link2="${tf_prefix}pillar_2" reason="Never"/>
+        <disable_collisions link1="${tf_prefix}RealSense_D405" link2="${tf_prefix}pillar_3" reason="Never"/>
+        <disable_collisions link1="${tf_prefix}RealSense_D405" link2="${tf_prefix}pillar_4" reason="Never"/>
+        <disable_collisions link1="${tf_prefix}RealSense_D405" link2="${tf_prefix}suction_mount" reason="Never"/>
+        <disable_collisions link1="${tf_prefix}RealSense_Holder_01" link2="${tf_prefix}pillar_1" reason="Never"/>
+        <disable_collisions link1="${tf_prefix}RealSense_Holder_01" link2="${tf_prefix}pillar_2" reason="Never"/>
+        <disable_collisions link1="${tf_prefix}RealSense_Holder_01" link2="${tf_prefix}pillar_3" reason="Never"/>
+        <disable_collisions link1="${tf_prefix}RealSense_Holder_01" link2="${tf_prefix}suction_mount" reason="Never"/>
+        <disable_collisions link1="${tf_prefix}RealSense_Holder_01" link2="${tf_prefix}tube" reason="Never"/>
+        <disable_collisions link1="${tf_prefix}Custom_Mount" link2="${tf_prefix}base_mount" reason="Never"/>
+        <disable_collisions link1="${tf_prefix}Custom_Mount" link2="${tf_prefix}pillar_1" reason="Never"/>
+        <disable_collisions link1="${tf_prefix}Custom_Mount" link2="${tf_prefix}pillar_2" reason="Never"/>
+        <disable_collisions link1="${tf_prefix}Custom_Mount" link2="${tf_prefix}pillar_3" reason="Never"/>
+        <disable_collisions link1="${tf_prefix}Custom_Mount" link2="${tf_prefix}pillar_4" reason="Never"/>
+        <disable_collisions link1="${tf_prefix}Custom_Mount" link2="${tf_prefix}suction_cup" reason="Never"/>
+        <disable_collisions link1="${tf_prefix}Custom_Mount" link2="${tf_prefix}suction_mount" reason="Never"/>
+        <disable_collisions link1="${tf_prefix}Custom_Mount" link2="${tf_prefix}tube" reason="Never"/>
+        <disable_collisions link1="${tf_prefix}base_mount" link2="${tf_prefix}pillar_1" reason="Adjacent"/>
+        <disable_collisions link1="${tf_prefix}base_mount" link2="${tf_prefix}pillar_2" reason="Default"/>
+        <disable_collisions link1="${tf_prefix}base_mount" link2="${tf_prefix}pillar_3" reason="Default"/>
+        <disable_collisions link1="${tf_prefix}base_mount" link2="${tf_prefix}pillar_4" reason="Adjacent"/>
+        <disable_collisions link1="${tf_prefix}base_mount" link2="${tf_prefix}suction_cup" reason="Never"/>
+        <disable_collisions link1="${tf_prefix}base_mount" link2="${tf_prefix}suction_mount" reason="Never"/>
+        <disable_collisions link1="${tf_prefix}base_mount" link2="${tf_prefix}tube" reason="Never"/>
+        <disable_collisions link1="${tf_prefix}carriage_left" link2="${tf_prefix}pillar_1" reason="Never"/>
+        <disable_collisions link1="${tf_prefix}carriage_left" link2="${tf_prefix}pillar_2" reason="Never"/>
+        <disable_collisions link1="${tf_prefix}carriage_left" link2="${tf_prefix}pillar_3" reason="Never"/>
+        <disable_collisions link1="${tf_prefix}carriage_left" link2="${tf_prefix}pillar_4" reason="Never"/>
+        <disable_collisions link1="${tf_prefix}carriage_left" link2="${tf_prefix}suction_cup" reason="Never"/>
+        <disable_collisions link1="${tf_prefix}carriage_left" link2="${tf_prefix}suction_mount" reason="Never"/>
+        <disable_collisions link1="${tf_prefix}carriage_left" link2="${tf_prefix}tube" reason="Never"/>
+        <disable_collisions link1="${tf_prefix}carriage_right" link2="${tf_prefix}pillar_1" reason="Never"/>
+        <disable_collisions link1="${tf_prefix}carriage_right" link2="${tf_prefix}pillar_2" reason="Never"/>
+        <disable_collisions link1="${tf_prefix}carriage_right" link2="${tf_prefix}pillar_3" reason="Never"/>
+        <disable_collisions link1="${tf_prefix}carriage_right" link2="${tf_prefix}pillar_4" reason="Never"/>
+        <disable_collisions link1="${tf_prefix}carriage_right" link2="${tf_prefix}suction_cup" reason="Never"/>
+        <disable_collisions link1="${tf_prefix}carriage_right" link2="${tf_prefix}suction_mount" reason="Never"/>
+        <disable_collisions link1="${tf_prefix}carriage_right" link2="${tf_prefix}tube" reason="Never"/>
+        <disable_collisions link1="${tf_prefix}gripper_left" link2="${tf_prefix}pillar_1" reason="Never"/>
+        <disable_collisions link1="${tf_prefix}gripper_left" link2="${tf_prefix}pillar_2" reason="Never"/>
+        <disable_collisions link1="${tf_prefix}gripper_left" link2="${tf_prefix}pillar_3" reason="Never"/>
+        <disable_collisions link1="${tf_prefix}gripper_left" link2="${tf_prefix}pillar_4" reason="Never"/>
+        <disable_collisions link1="${tf_prefix}gripper_left" link2="${tf_prefix}suction_cup" reason="Never"/>
+        <disable_collisions link1="${tf_prefix}gripper_left" link2="${tf_prefix}suction_mount" reason="Never"/>
+        <disable_collisions link1="${tf_prefix}gripper_left" link2="${tf_prefix}tube" reason="Never"/>
+        <disable_collisions link1="${tf_prefix}gripper_right" link2="${tf_prefix}pillar_1" reason="Never"/>
+        <disable_collisions link1="${tf_prefix}gripper_right" link2="${tf_prefix}pillar_2" reason="Never"/>
+        <disable_collisions link1="${tf_prefix}gripper_right" link2="${tf_prefix}pillar_3" reason="Never"/>
+        <disable_collisions link1="${tf_prefix}gripper_right" link2="${tf_prefix}pillar_4" reason="Never"/>
+        <disable_collisions link1="${tf_prefix}gripper_right" link2="${tf_prefix}suction_cup" reason="Never"/>
+        <disable_collisions link1="${tf_prefix}gripper_right" link2="${tf_prefix}suction_mount" reason="Never"/>
+        <disable_collisions link1="${tf_prefix}gripper_right" link2="${tf_prefix}tube" reason="Never"/>
+        <disable_collisions link1="${tf_prefix}link_3" link2="${tf_prefix}pillar_3" reason="Never"/>
+        <disable_collisions link1="${tf_prefix}link_3" link2="${tf_prefix}pillar_4" reason="Never"/>
+        <disable_collisions link1="${tf_prefix}link_4" link2="${tf_prefix}link_5" reason="Adjacent"/>
+        <disable_collisions link1="${tf_prefix}link_4" link2="${tf_prefix}link_6" reason="Never"/>
+        <disable_collisions link1="${tf_prefix}link_5" link2="${tf_prefix}link_6" reason="Adjacent"/>
+        <disable_collisions link1="${tf_prefix}link_5" link2="${tf_prefix}pillar_1" reason="Never"/>
+        <disable_collisions link1="${tf_prefix}link_5" link2="${tf_prefix}pillar_2" reason="Never"/>
+        <disable_collisions link1="${tf_prefix}link_5" link2="${tf_prefix}pillar_3" reason="Never"/>
+        <disable_collisions link1="${tf_prefix}link_5" link2="${tf_prefix}pillar_4" reason="Never"/>
+        <disable_collisions link1="${tf_prefix}link_5" link2="${tf_prefix}suction_cup" reason="Never"/>
+        <disable_collisions link1="${tf_prefix}link_5" link2="${tf_prefix}suction_mount" reason="Never"/>
+        <disable_collisions link1="${tf_prefix}link_5" link2="${tf_prefix}tube" reason="Never"/>
+        <disable_collisions link1="${tf_prefix}link_6" link2="${tf_prefix}pillar_1" reason="Never"/>
+        <disable_collisions link1="${tf_prefix}link_6" link2="${tf_prefix}pillar_2" reason="Never"/>
+        <disable_collisions link1="${tf_prefix}link_6" link2="${tf_prefix}pillar_3" reason="Never"/>
+        <disable_collisions link1="${tf_prefix}link_6" link2="${tf_prefix}pillar_4" reason="Never"/>
+        <disable_collisions link1="${tf_prefix}link_6" link2="${tf_prefix}suction_cup" reason="Never"/>
+        <disable_collisions link1="${tf_prefix}link_6" link2="${tf_prefix}suction_mount" reason="Never"/>
+        <disable_collisions link1="${tf_prefix}link_6" link2="${tf_prefix}tube" reason="Never"/>
+        <disable_collisions link1="${tf_prefix}pillar_1" link2="${tf_prefix}pillar_2" reason="Never"/>
+        <disable_collisions link1="${tf_prefix}pillar_1" link2="${tf_prefix}pillar_3" reason="Never"/>
+        <disable_collisions link1="${tf_prefix}pillar_1" link2="${tf_prefix}pillar_4" reason="Never"/>
+        <disable_collisions link1="${tf_prefix}pillar_1" link2="${tf_prefix}suction_cup" reason="Never"/>
+        <disable_collisions link1="${tf_prefix}pillar_1" link2="${tf_prefix}suction_mount" reason="Adjacent"/>
+        <disable_collisions link1="${tf_prefix}pillar_1" link2="${tf_prefix}tube" reason="Never"/>
+        <disable_collisions link1="${tf_prefix}pillar_2" link2="${tf_prefix}pillar_3" reason="Never"/>
+        <disable_collisions link1="${tf_prefix}pillar_2" link2="${tf_prefix}pillar_4" reason="Never"/>
+        <disable_collisions link1="${tf_prefix}pillar_2" link2="${tf_prefix}suction_cup" reason="Never"/>
+        <disable_collisions link1="${tf_prefix}pillar_2" link2="${tf_prefix}suction_mount" reason="Adjacent"/>
+        <disable_collisions link1="${tf_prefix}pillar_2" link2="${tf_prefix}tube" reason="Never"/>
+        <disable_collisions link1="${tf_prefix}pillar_3" link2="${tf_prefix}pillar_4" reason="Never"/>
+        <disable_collisions link1="${tf_prefix}pillar_3" link2="${tf_prefix}suction_cup" reason="Never"/>
+        <disable_collisions link1="${tf_prefix}pillar_3" link2="${tf_prefix}suction_mount" reason="Adjacent"/>
+        <disable_collisions link1="${tf_prefix}pillar_3" link2="${tf_prefix}tube" reason="Never"/>
+        <disable_collisions link1="${tf_prefix}pillar_4" link2="${tf_prefix}suction_cup" reason="Never"/>
+        <disable_collisions link1="${tf_prefix}pillar_4" link2="${tf_prefix}suction_mount" reason="Default"/>
+        <disable_collisions link1="${tf_prefix}pillar_4" link2="${tf_prefix}tube" reason="Never"/>
+        <disable_collisions link1="${tf_prefix}suction_cup" link2="${tf_prefix}suction_mount" reason="Adjacent"/>
+        <disable_collisions link1="${tf_prefix}suction_cup" link2="${tf_prefix}tube" reason="Adjacent"/>
+        <disable_collisions link1="${tf_prefix}suction_mount" link2="${tf_prefix}tube" reason="Never"/>
+    </xacro:if>
     <xacro:if value="${srdf_use_downdraft}">
         <disable_collisions link1="${tf_prefix}Back_Plate_Exhaust" link2="${tf_prefix}Bottom_Box" reason="Never"/>
@@ -138,13 +283,5 @@
         <disable_collisions link1="${tf_prefix}Back_Plate_Exhaust" link2="${tf_prefix}Top_Camera_frame" reason="Never"/>
         <disable_collisions link1="${tf_prefix}Custom_Mount" link2="${tf_prefix}Side_Plates_Right" reason="Never"/>
-        <disable_collisions link1="${tf_prefix}Custom_Mount" link2="${tf_prefix}base_mount" reason="Never"/>
         <disable_collisions link1="${tf_prefix}Custom_Mount" link2="${tf_prefix}light_1" reason="Never"/>
-        <disable_collisions link1="${tf_prefix}Custom_Mount" link2="${tf_prefix}pillar_1" reason="Never"/>
-        <disable_collisions link1="${tf_prefix}Custom_Mount" link2="${tf_prefix}pillar_2" reason="Never"/>
-        <disable_collisions link1="${tf_prefix}Custom_Mount" link2="${tf_prefix}pillar_3" reason="Never"/>
-        <disable_collisions link1="${tf_prefix}Custom_Mount" link2="${tf_prefix}pillar_4" reason="Never"/>
-        <disable_collisions link1="${tf_prefix}Custom_Mount" link2="${tf_prefix}suction_cup" reason="Never"/>
-        <disable_collisions link1="${tf_prefix}Custom_Mount" link2="${tf_prefix}suction_mount" reason="Never"/>
-        <disable_collisions link1="${tf_prefix}Custom_Mount" link2="${tf_prefix}tube" reason="Never"/>
         <disable_collisions link1="${tf_prefix}Back_Plate_Exhaust" link2="${tf_prefix}Front_Weld_Plate" reason="Never"/>
         <disable_collisions link1="${tf_prefix}Back_Plate_Exhaust" link2="${tf_prefix}Letter_Trimmer_Holder" reason="Never"/>
@@ -176,11 +313,4 @@
         <disable_collisions link1="${tf_prefix}Back_Plate_Exhaust" link2="${tf_prefix}link_5" reason="Never"/>
         <disable_collisions link1="${tf_prefix}Back_Plate_Exhaust" link2="${tf_prefix}link_6" reason="Never"/>
-        <disable_collisions link1="${tf_prefix}Back_Plate_Exhaust" link2="${tf_prefix}pillar_1" reason="Never"/>
-        <disable_collisions link1="${tf_prefix}Back_Plate_Exhaust" link2="${tf_prefix}pillar_2" reason="Never"/>
-        <disable_collisions link1="${tf_prefix}Back_Plate_Exhaust" link2="${tf_prefix}pillar_3" reason="Never"/>
-        <disable_collisions link1="${tf_prefix}Back_Plate_Exhaust" link2="${tf_prefix}pillar_4" reason="Never"/>
-        <disable_collisions link1="${tf_prefix}Back_Plate_Exhaust" link2="${tf_prefix}suction_cup" reason="Never"/>
-        <disable_collisions link1="${tf_prefix}Back_Plate_Exhaust" link2="${tf_prefix}suction_mount" reason="Never"/>
-        <disable_collisions link1="${tf_prefix}Back_Plate_Exhaust" link2="${tf_prefix}tube" reason="Never"/>
         <disable_collisions link1="${tf_prefix}Bottom_Box" link2="${tf_prefix}Chute_01" reason="Never"/>
         <disable_collisions link1="${tf_prefix}Bottom_Box" link2="${tf_prefix}Chute_02" reason="Never"/>
@@ -384,11 +514,6 @@
         <disable_collisions link1="${tf_prefix}RealSense_D405" link2="${tf_prefix}link_2" reason="Never"/>
         <disable_collisions link1="${tf_prefix}RealSense_D405" link2="${tf_prefix}link_3" reason="Never"/>
-        <disable_collisions link1="${tf_prefix}RealSense_D405" link2="${tf_prefix}pillar_1" reason="Never"/>
-        <disable_collisions link1="${tf_prefix}RealSense_D405" link2="${tf_prefix}pillar_2" reason="Never"/>
-        <disable_collisions link1="${tf_prefix}RealSense_D405" link2="${tf_prefix}pillar_3" reason="Never"/>
-        <disable_collisions link1="${tf_prefix}RealSense_D405" link2="${tf_prefix}pillar_4" reason="Never"/>
-        <disable_collisions link1="${tf_prefix}RealSense_D405" link2="${tf_prefix}suction_mount" reason="Never"/>
         <disable_collisions link1="${tf_prefix}RealSense_D405" link2="${tf_prefix}Top_Camera_frame" reason="Never"/>
-        <disable_collisions link1="${tf_prefix}RealSense_D405" link2="${tf_prefix}tube" reason="Never"/>
+        <disable_collisions link1="${tf_prefix}RealSense_Holder_01" link2="${tf_prefix}Top_Camera_frame" reason="Never"/>
         <disable_collisions link1="${tf_prefix}RealSense_Holder_01" link2="${tf_prefix}RealSense_Holder_02" reason="Adjacent"/>
         <disable_collisions link1="${tf_prefix}RealSense_Holder_01" link2="${tf_prefix}Rear_Panel" reason="Never"/>
@@ -406,10 +531,4 @@
         <disable_collisions link1="${tf_prefix}RealSense_Holder_01" link2="${tf_prefix}link_2" reason="Never"/>
         <disable_collisions link1="${tf_prefix}RealSense_Holder_01" link2="${tf_prefix}link_3" reason="Never"/>
-        <disable_collisions link1="${tf_prefix}RealSense_Holder_01" link2="${tf_prefix}pillar_1" reason="Never"/>
-        <disable_collisions link1="${tf_prefix}RealSense_Holder_01" link2="${tf_prefix}pillar_2" reason="Never"/>
-        <disable_collisions link1="${tf_prefix}RealSense_Holder_01" link2="${tf_prefix}Top_Camera_frame" reason="Never"/>
-        <disable_collisions link1="${tf_prefix}RealSense_Holder_01" link2="${tf_prefix}pillar_3" reason="Never"/>
-        <disable_collisions link1="${tf_prefix}RealSense_Holder_01" link2="${tf_prefix}suction_mount" reason="Never"/>
-        <disable_collisions link1="${tf_prefix}RealSense_Holder_01" link2="${tf_prefix}tube" reason="Never"/>
         <disable_collisions link1="${tf_prefix}RealSense_Holder_02" link2="${tf_prefix}Rear_Panel" reason="Never"/>
         <disable_collisions link1="${tf_prefix}RealSense_Holder_02" link2="${tf_prefix}Side_Plates_Left" reason="Never"/>
@@ -428,7 +547,4 @@
         <disable_collisions link1="${tf_prefix}RealSense_Holder_02" link2="${tf_prefix}link_4" reason="Never"/>
         <disable_collisions link1="${tf_prefix}RealSense_Holder_02" link2="${tf_prefix}link_5" reason="Never"/>
-        <disable_collisions link1="${tf_prefix}RealSense_Holder_02" link2="${tf_prefix}pillar_1" reason="Never"/>
-        <disable_collisions link1="${tf_prefix}RealSense_Holder_02" link2="${tf_prefix}pillar_3" reason="Never"/>
-        <disable_collisions link1="${tf_prefix}RealSense_Holder_02" link2="${tf_prefix}tube" reason="Never"/>
         <disable_collisions link1="${tf_prefix}RealSense_Holder_02" link2="${tf_prefix}Top_Camera_frame" reason="Never"/>
         <disable_collisions link1="${tf_prefix}Rear_Panel" link2="${tf_prefix}Side_Plates_Left" reason="Default"/>
@@ -446,10 +562,5 @@
         <disable_collisions link1="${tf_prefix}Rear_Panel" link2="${tf_prefix}link_3" reason="Never"/>
         <disable_collisions link1="${tf_prefix}Rear_Panel" link2="${tf_prefix}link_5" reason="Never"/>
-        <disable_collisions link1="${tf_prefix}Rear_Panel" link2="${tf_prefix}pillar_1" reason="Never"/>
-        <disable_collisions link1="${tf_prefix}Rear_Panel" link2="${tf_prefix}pillar_2" reason="Never"/>
-        <disable_collisions link1="${tf_prefix}Rear_Panel" link2="${tf_prefix}pillar_3" reason="Never"/>
-        <disable_collisions link1="${tf_prefix}Rear_Panel" link2="${tf_prefix}pillar_4" reason="Never"/>
         <disable_collisions link1="${tf_prefix}Rear_Panel" link2="${tf_prefix}Top_Camera_frame" reason="Never"/>
-        <disable_collisions link1="${tf_prefix}Rear_Panel" link2="${tf_prefix}tube" reason="Never"/>
         <disable_collisions link1="${tf_prefix}Side_Plates_Left" link2="${tf_prefix}Side_Plates_Right" reason="Never"/>
         <disable_collisions link1="${tf_prefix}Side_Plates_Left" link2="${tf_prefix}Top_Panel" reason="Adjacent"/>
@@ -481,12 +592,5 @@
         <disable_collisions link1="${tf_prefix}Side_Plates_Right" link2="${tf_prefix}link_5" reason="Never"/>
         <disable_collisions link1="${tf_prefix}Side_Plates_Right" link2="${tf_prefix}link_6" reason="Never"/>
-        <disable_collisions link1="${tf_prefix}Side_Plates_Right" link2="${tf_prefix}pillar_1" reason="Never"/>
-        <disable_collisions link1="${tf_prefix}Side_Plates_Right" link2="${tf_prefix}pillar_2" reason="Never"/>
-        <disable_collisions link1="${tf_prefix}Side_Plates_Right" link2="${tf_prefix}pillar_3" reason="Never"/>
-        <disable_collisions link1="${tf_prefix}Side_Plates_Right" link2="${tf_prefix}pillar_4" reason="Never"/>
-        <disable_collisions link1="${tf_prefix}Side_Plates_Right" link2="${tf_prefix}suction_cup" reason="Never"/>
         <disable_collisions link1="${tf_prefix}Side_Plates_Right" link2="${tf_prefix}Top_Camera_frame" reason="Default"/>
-        <disable_collisions link1="${tf_prefix}Side_Plates_Right" link2="${tf_prefix}suction_mount" reason="Never"/>
-        <disable_collisions link1="${tf_prefix}Side_Plates_Right" link2="${tf_prefix}tube" reason="Never"/>
         <disable_collisions link1="${tf_prefix}Top_Panel" link2="${tf_prefix}Top_Weld_Plate" reason="Never"/>
         <disable_collisions link1="${tf_prefix}Top_Panel" link2="${tf_prefix}Vibration_Table_Plate" reason="Adjacent"/>
@@ -514,9 +618,4 @@
         <disable_collisions link1="${tf_prefix}Top_Weld_Plate" link2="${tf_prefix}link_4" reason="Never"/>
         <disable_collisions link1="${tf_prefix}Top_Weld_Plate" link2="${tf_prefix}link_5" reason="Never"/>
-        <disable_collisions link1="${tf_prefix}Top_Weld_Plate" link2="${tf_prefix}pillar_1" reason="Never"/>
-        <disable_collisions link1="${tf_prefix}Top_Weld_Plate" link2="${tf_prefix}pillar_2" reason="Never"/>
-        <disable_collisions link1="${tf_prefix}Top_Weld_Plate" link2="${tf_prefix}pillar_4" reason="Never"/>
-        <disable_collisions link1="${tf_prefix}Top_Weld_Plate" link2="${tf_prefix}suction_mount" reason="Never"/>
-        <disable_collisions link1="${tf_prefix}Top_Weld_Plate" link2="${tf_prefix}tube" reason="Never"/>
         <disable_collisions link1="${tf_prefix}Vibration_Table_Plate" link2="${tf_prefix}Vibration_Table_Top_Plate" reason="Adjacent"/>
         <disable_collisions link1="${tf_prefix}Vibration_Table_Plate" link2="${tf_prefix}base_link" reason="Never"/>
@@ -544,11 +643,4 @@
         <disable_collisions link1="${tf_prefix}base_mount" link2="${tf_prefix}link_5" reason="Default"/>
         <disable_collisions link1="${tf_prefix}base_mount" link2="${tf_prefix}link_6" reason="Adjacent"/>
-        <disable_collisions link1="${tf_prefix}base_mount" link2="${tf_prefix}pillar_1" reason="Adjacent"/>
-        <disable_collisions link1="${tf_prefix}base_mount" link2="${tf_prefix}pillar_2" reason="Default"/>
-        <disable_collisions link1="${tf_prefix}base_mount" link2="${tf_prefix}pillar_3" reason="Default"/>
-        <disable_collisions link1="${tf_prefix}base_mount" link2="${tf_prefix}pillar_4" reason="Adjacent"/>
-        <disable_collisions link1="${tf_prefix}base_mount" link2="${tf_prefix}suction_cup" reason="Never"/>
-        <disable_collisions link1="${tf_prefix}base_mount" link2="${tf_prefix}suction_mount" reason="Never"/>
-        <disable_collisions link1="${tf_prefix}base_mount" link2="${tf_prefix}tube" reason="Never"/>
         <disable_collisions link1="${tf_prefix}carriage_left" link2="${tf_prefix}carriage_right" reason="Never"/>
         <disable_collisions link1="${tf_prefix}carriage_left" link2="${tf_prefix}gripper_left" reason="Adjacent"/>
@@ -559,11 +651,4 @@
         <disable_collisions link1="${tf_prefix}carriage_left" link2="${tf_prefix}link_5" reason="Never"/>
         <disable_collisions link1="${tf_prefix}carriage_left" link2="${tf_prefix}link_6" reason="Adjacent"/>
-        <disable_collisions link1="${tf_prefix}carriage_left" link2="${tf_prefix}pillar_1" reason="Never"/>
-        <disable_collisions link1="${tf_prefix}carriage_left" link2="${tf_prefix}pillar_2" reason="Never"/>
-        <disable_collisions link1="${tf_prefix}carriage_left" link2="${tf_prefix}pillar_3" reason="Never"/>
-        <disable_collisions link1="${tf_prefix}carriage_left" link2="${tf_prefix}pillar_4" reason="Never"/>
-        <disable_collisions link1="${tf_prefix}carriage_left" link2="${tf_prefix}suction_cup" reason="Never"/>
-        <disable_collisions link1="${tf_prefix}carriage_left" link2="${tf_prefix}suction_mount" reason="Never"/>
-        <disable_collisions link1="${tf_prefix}carriage_left" link2="${tf_prefix}tube" reason="Never"/>
         <disable_collisions link1="${tf_prefix}carriage_right" link2="${tf_prefix}gripper_left" reason="Never"/>
         <disable_collisions link1="${tf_prefix}carriage_right" link2="${tf_prefix}gripper_right" reason="Adjacent"/>
@@ -573,11 +658,4 @@
         <disable_collisions link1="${tf_prefix}carriage_right" link2="${tf_prefix}link_5" reason="Never"/>
         <disable_collisions link1="${tf_prefix}carriage_right" link2="${tf_prefix}link_6" reason="Adjacent"/>
-        <disable_collisions link1="${tf_prefix}carriage_right" link2="${tf_prefix}pillar_1" reason="Never"/>
-        <disable_collisions link1="${tf_prefix}carriage_right" link2="${tf_prefix}pillar_2" reason="Never"/>
-        <disable_collisions link1="${tf_prefix}carriage_right" link2="${tf_prefix}pillar_3" reason="Never"/>
-        <disable_collisions link1="${tf_prefix}carriage_right" link2="${tf_prefix}pillar_4" reason="Never"/>
-        <disable_collisions link1="${tf_prefix}carriage_right" link2="${tf_prefix}suction_cup" reason="Never"/>
-        <disable_collisions link1="${tf_prefix}carriage_right" link2="${tf_prefix}suction_mount" reason="Never"/>
-        <disable_collisions link1="${tf_prefix}carriage_right" link2="${tf_prefix}tube" reason="Never"/>
         <disable_collisions link1="${tf_prefix}gripper_left" link2="${tf_prefix}gripper_right" reason="Never"/>
         <disable_collisions link1="${tf_prefix}gripper_left" link2="${tf_prefix}light_1" reason="Never"/>
@@ -586,11 +664,4 @@
         <disable_collisions link1="${tf_prefix}gripper_left" link2="${tf_prefix}link_5" reason="Never"/>
         <disable_collisions link1="${tf_prefix}gripper_left" link2="${tf_prefix}link_6" reason="Never"/>
-        <disable_collisions link1="${tf_prefix}gripper_left" link2="${tf_prefix}pillar_1" reason="Never"/>
-        <disable_collisions link1="${tf_prefix}gripper_left" link2="${tf_prefix}pillar_2" reason="Never"/>
-        <disable_collisions link1="${tf_prefix}gripper_left" link2="${tf_prefix}pillar_3" reason="Never"/>
-        <disable_collisions link1="${tf_prefix}gripper_left" link2="${tf_prefix}pillar_4" reason="Never"/>
-        <disable_collisions link1="${tf_prefix}gripper_left" link2="${tf_prefix}suction_cup" reason="Never"/>
-        <disable_collisions link1="${tf_prefix}gripper_left" link2="${tf_prefix}suction_mount" reason="Never"/>
-        <disable_collisions link1="${tf_prefix}gripper_left" link2="${tf_prefix}tube" reason="Never"/>
         <disable_collisions link1="${tf_prefix}gripper_right" link2="${tf_prefix}light_1" reason="Never"/>
         <disable_collisions link1="${tf_prefix}gripper_right" link2="${tf_prefix}link_3" reason="Never"/>
@@ -598,11 +669,4 @@
         <disable_collisions link1="${tf_prefix}gripper_right" link2="${tf_prefix}link_5" reason="Never"/>
         <disable_collisions link1="${tf_prefix}gripper_right" link2="${tf_prefix}link_6" reason="Never"/>
-        <disable_collisions link1="${tf_prefix}gripper_right" link2="${tf_prefix}pillar_1" reason="Never"/>
-        <disable_collisions link1="${tf_prefix}gripper_right" link2="${tf_prefix}pillar_2" reason="Never"/>
-        <disable_collisions link1="${tf_prefix}gripper_right" link2="${tf_prefix}pillar_3" reason="Never"/>
-        <disable_collisions link1="${tf_prefix}gripper_right" link2="${tf_prefix}pillar_4" reason="Never"/>
-        <disable_collisions link1="${tf_prefix}gripper_right" link2="${tf_prefix}suction_cup" reason="Never"/>
-        <disable_collisions link1="${tf_prefix}gripper_right" link2="${tf_prefix}suction_mount" reason="Never"/>
-        <disable_collisions link1="${tf_prefix}gripper_right" link2="${tf_prefix}tube" reason="Never"/>
         <disable_collisions link1="${tf_prefix}light_1" link2="${tf_prefix}light_2" reason="Never"/>
         <disable_collisions link1="${tf_prefix}light_1" link2="${tf_prefix}link_1" reason="Never"/>
@@ -612,22 +676,4 @@
         <disable_collisions link1="${tf_prefix}light_1" link2="${tf_prefix}link_5" reason="Never"/>
         <disable_collisions link1="${tf_prefix}light_1" link2="${tf_prefix}link_6" reason="Never"/>
-        <disable_collisions link1="${tf_prefix}light_1" link2="${tf_prefix}pillar_1" reason="Never"/>
-        <disable_collisions link1="${tf_prefix}light_1" link2="${tf_prefix}pillar_2" reason="Never"/>
-        <disable_collisions link1="${tf_prefix}light_1" link2="${tf_prefix}pillar_3" reason="Never"/>
-        <disable_collisions link1="${tf_prefix}light_1" link2="${tf_prefix}pillar_4" reason="Never"/>
-        <disable_collisions link1="${tf_prefix}light_1" link2="${tf_prefix}suction_cup" reason="Never"/>
-        <disable_collisions link1="${tf_prefix}light_1" link2="${tf_prefix}suction_mount" reason="Never"/>
-        <disable_collisions link1="${tf_prefix}light_1" link2="${tf_prefix}tube" reason="Never"/>
-        <disable_collisions link1="${tf_prefix}light_2" link2="${tf_prefix}link_1" reason="Never"/>
-        <disable_collisions link1="${tf_prefix}light_2" link2="${tf_prefix}link_2" reason="Never"/>
-        <disable_collisions link1="${tf_prefix}light_2" link2="${tf_prefix}link_3" reason="Never"/>
-        <disable_collisions link1="${tf_prefix}light_2" link2="${tf_prefix}link_4" reason="Never"/>
-        <disable_collisions link1="${tf_prefix}light_2" link2="${tf_prefix}link_5" reason="Never"/>
-        <disable_collisions link1="${tf_prefix}light_2" link2="${tf_prefix}pillar_1" reason="Never"/>
-        <disable_collisions link1="${tf_prefix}light_2" link2="${tf_prefix}pillar_2" reason="Never"/>
-        <disable_collisions link1="${tf_prefix}light_2" link2="${tf_prefix}pillar_3" reason="Never"/>
-        <disable_collisions link1="${tf_prefix}light_2" link2="${tf_prefix}pillar_4" reason="Never"/>
-        <disable_collisions link1="${tf_prefix}light_2" link2="${tf_prefix}suction_mount" reason="Never"/>
-        <disable_collisions link1="${tf_prefix}light_2" link2="${tf_prefix}tube" reason="Never"/>
         <disable_collisions link1="${tf_prefix}link_1" link2="${tf_prefix}link_2" reason="Adjacent"/>
         <disable_collisions link1="${tf_prefix}link_2" link2="${tf_prefix}link_3" reason="Adjacent"/>
@@ -635,44 +681,4 @@
         <disable_collisions link1="${tf_prefix}link_3" link2="${tf_prefix}link_5" reason="Never"/>
         <disable_collisions link1="${tf_prefix}link_3" link2="${tf_prefix}link_6" reason="Never"/>
-        <disable_collisions link1="${tf_prefix}link_3" link2="${tf_prefix}pillar_3" reason="Never"/>
-        <disable_collisions link1="${tf_prefix}link_3" link2="${tf_prefix}pillar_4" reason="Never"/>
-        <disable_collisions link1="${tf_prefix}link_4" link2="${tf_prefix}link_5" reason="Adjacent"/>
-        <disable_collisions link1="${tf_prefix}link_4" link2="${tf_prefix}link_6" reason="Never"/>
-        <disable_collisions link1="${tf_prefix}link_5" link2="${tf_prefix}link_6" reason="Adjacent"/>
-        <disable_collisions link1="${tf_prefix}link_5" link2="${tf_prefix}pillar_1" reason="Never"/>
-        <disable_collisions link1="${tf_prefix}link_5" link2="${tf_prefix}pillar_2" reason="Never"/>
-        <disable_collisions link1="${tf_prefix}link_5" link2="${tf_prefix}pillar_3" reason="Never"/>
-        <disable_collisions link1="${tf_prefix}link_5" link2="${tf_prefix}pillar_4" reason="Never"/>
-        <disable_collisions link1="${tf_prefix}link_5" link2="${tf_prefix}suction_cup" reason="Never"/>
-        <disable_collisions link1="${tf_prefix}link_5" link2="${tf_prefix}suction_mount" reason="Never"/>
-        <disable_collisions link1="${tf_prefix}link_5" link2="${tf_prefix}tube" reason="Never"/>
-        <disable_collisions link1="${tf_prefix}link_6" link2="${tf_prefix}pillar_1" reason="Never"/>
-        <disable_collisions link1="${tf_prefix}link_6" link2="${tf_prefix}pillar_2" reason="Never"/>
-        <disable_collisions link1="${tf_prefix}link_6" link2="${tf_prefix}pillar_3" reason="Never"/>
-        <disable_collisions link1="${tf_prefix}link_6" link2="${tf_prefix}pillar_4" reason="Never"/>
-        <disable_collisions link1="${tf_prefix}link_6" link2="${tf_prefix}suction_cup" reason="Never"/>
-        <disable_collisions link1="${tf_prefix}link_6" link2="${tf_prefix}suction_mount" reason="Never"/>
-        <disable_collisions link1="${tf_prefix}link_6" link2="${tf_prefix}tube" reason="Never"/>
-        <disable_collisions link1="${tf_prefix}pillar_1" link2="${tf_prefix}pillar_2" reason="Never"/>
-        <disable_collisions link1="${tf_prefix}pillar_1" link2="${tf_prefix}pillar_3" reason="Never"/>
-        <disable_collisions link1="${tf_prefix}pillar_1" link2="${tf_prefix}pillar_4" reason="Never"/>
-        <disable_collisions link1="${tf_prefix}pillar_1" link2="${tf_prefix}suction_cup" reason="Never"/>
-        <disable_collisions link1="${tf_prefix}pillar_1" link2="${tf_prefix}suction_mount" reason="Adjacent"/>
-        <disable_collisions link1="${tf_prefix}pillar_1" link2="${tf_prefix}tube" reason="Never"/>
-        <disable_collisions link1="${tf_prefix}pillar_2" link2="${tf_prefix}pillar_3" reason="Never"/>
-        <disable_collisions link1="${tf_prefix}pillar_2" link2="${tf_prefix}pillar_4" reason="Never"/>
-        <disable_collisions link1="${tf_prefix}pillar_2" link2="${tf_prefix}suction_cup" reason="Never"/>
-        <disable_collisions link1="${tf_prefix}pillar_2" link2="${tf_prefix}suction_mount" reason="Adjacent"/>
-        <disable_collisions link1="${tf_prefix}pillar_2" link2="${tf_prefix}tube" reason="Never"/>
-        <disable_collisions link1="${tf_prefix}pillar_3" link2="${tf_prefix}pillar_4" reason="Never"/>
-        <disable_collisions link1="${tf_prefix}pillar_3" link2="${tf_prefix}suction_cup" reason="Never"/>
-        <disable_collisions link1="${tf_prefix}pillar_3" link2="${tf_prefix}suction_mount" reason="Adjacent"/>
-        <disable_collisions link1="${tf_prefix}pillar_3" link2="${tf_prefix}tube" reason="Never"/>
-        <disable_collisions link1="${tf_prefix}pillar_4" link2="${tf_prefix}suction_cup" reason="Never"/>
-        <disable_collisions link1="${tf_prefix}pillar_4" link2="${tf_prefix}suction_mount" reason="Default"/>
-        <disable_collisions link1="${tf_prefix}pillar_4" link2="${tf_prefix}tube" reason="Never"/>
-        <disable_collisions link1="${tf_prefix}suction_cup" link2="${tf_prefix}suction_mount" reason="Adjacent"/>
-        <disable_collisions link1="${tf_prefix}suction_cup" link2="${tf_prefix}tube" reason="Adjacent"/>
-        <disable_collisions link1="${tf_prefix}suction_mount" link2="${tf_prefix}tube" reason="Never"/>
     </xacro:if>
     <xacro:if value="${arm_variant == 'follower'}">
