Commit message: Fixed collissions

File: trossen_arm_moveit/config/wxai.srdf.xacro (robot description, xacro)
@@ -80,6 +80,6 @@
     </group_state>
     <group_state name="open" group="gripper">
-        <joint name="${tf_prefix}left_carriage_joint" value="0.044"/>
-        <joint name="${tf_prefix}right_carriage_joint" value="0.044"/>
+        <joint name="${tf_prefix}left_carriage_joint" value="0.022"/>
+        <joint name="${tf_prefix}right_carriage_joint" value="0.022"/>
     </group_state>
     <!--END EFFECTOR: Purpose: Represent information about an end effector.-->
