Commit message: changed the launch file for armor kit

File: trossen_arm_moveit/config/wxai.srdf.xacro (robot description, xacro)
@@ -64,4 +64,8 @@
     </group_state>
     <group_state name="open" group="gripper">
+        <joint name="${tf_prefix}left_carriage_joint" value="0.044"/>
+        <joint name="${tf_prefix}right_carriage_joint" value="0.044"/>
+    </group_state>
+    <group_state name="half_open" group="gripper">
         <joint name="${tf_prefix}left_carriage_joint" value="0.022"/>
         <joint name="${tf_prefix}right_carriage_joint" value="0.022"/>
@@ -72,14 +76,4 @@
     <disable_collisions link1="${tf_prefix}base_link" link2="${tf_prefix}link_1" reason="Adjacent"/>
     <disable_collisions link1="${tf_prefix}{tf_prefix}base_link" link2="${tf_prefix}link_2" reason="Never"/>
-    <!-- <disable_collisions link1="${tf_prefix}Custom_Mount" link2="${tf_prefix}link_1" reason="Default"/>
-    <disable_collisions link1="${tf_prefix}Custom_Mount" link2="${tf_prefix}link_2" reason="Default"/>
-    <disable_collisions link1="${tf_prefix}Custom_Mount" link2="${tf_prefix}link_5" reason="Default"/>
-    <disable_collisions link1="${tf_prefix}Custom_Mount" link2="${tf_prefix}link_6" reason="Adjacent"/>
-    <disable_collisions link1="${tf_prefix}Custom_Mount" link2="${tf_prefix}base_link" reason="Default"/>
-    <disable_collisions link1="${tf_prefix}Custom_Mount" link2="${tf_prefix}base_mount" reason="Never"/>
-    <disable_collisions link1="${tf_prefix}Custom_Mount" link2="${tf_prefix}carriage_left" reason="Never"/>
-    <disable_collisions link1="${tf_prefix}Custom_Mount" link2="${tf_prefix}carriage_right" reason="Never"/>
-    <disable_collisions link1="${tf_prefix}Custom_Mount" link2="${tf_prefix}gripper_left" reason="Never"/>
-    <disable_collisions link1="${tf_prefix}Custom_Mount" link2="${tf_prefix}gripper_right" reason="Never"/> -->
     <disable_collisions link1="${tf_prefix}carriage_left" link2="${tf_prefix}carriage_right" reason="Never"/>
     <disable_collisions link1="${tf_prefix}carriage_left" link2="${tf_prefix}gripper_left" reason="Adjacent"/>
@@ -132,5 +126,4 @@
     <disable_collisions link1="${tf_prefix}RealSense_Holder_01" link2="${tf_prefix}link_5" reason="Never"/>
     <disable_collisions link1="${tf_prefix}RealSense_Holder_01" link2="${tf_prefix}link_6" reason="Never"/>
-    <!-- <disable_collisions link1="${tf_prefix}Custom_Mount" link2="${tf_prefix}RealSense_Holder_02" reason="Never"/> -->
     <disable_collisions link1="${tf_prefix}RealSense_Holder_02" link2="${tf_prefix}base_link" reason="Never"/>
     <disable_collisions link1="${tf_prefix}RealSense_Holder_02" link2="${tf_prefix}carriage_left" reason="Never"/>
@@ -153,11 +146,4 @@
         <disable_collisions link1="${tf_prefix}Back_Plate_Exhaust" link2="${tf_prefix}suction_mount" reason="Never"/>
         <disable_collisions link1="${tf_prefix}Back_Plate_Exhaust" link2="${tf_prefix}tube" reason="Never"/>
-        <!-- <disable_collisions link1="${tf_prefix}Custom_Mount" link2="${tf_prefix}pillar_1" reason="Never"/>
-        <disable_collisions link1="${tf_prefix}Custom_Mount" link2="${tf_prefix}pillar_2" reason="Never"/>
-        <disable_collisions link1="${tf_prefix}Custom_Mount" link2="${tf_prefix}pillar_3" reason="Never"/>
-        <disable_collisions link1="${tf_prefix}Custom_Mount" link2="${tf_prefix}pillar_4" reason="Never"/>
-        <disable_collisions link1="${tf_prefix}Custom_Mount" link2="${tf_prefix}suction_cup" reason="Never"/>
-        <disable_collisions link1="${tf_prefix}Custom_Mount" link2="${tf_prefix}suction_mount" reason="Never"/>
-        <disable_collisions link1="${tf_prefix}Custom_Mount" link2="${tf_prefix}tube" reason="Never"/> -->
         <disable_collisions link1="${tf_prefix}Front_Weld_Plate" link2="${tf_prefix}suction_cup" reason="Default"/>
         <disable_collisions link1="${tf_prefix}Front_Weld_Plate" link2="${tf_prefix}suction_mount" reason="Default"/>
@@ -590,6 +576,6 @@
     </xacro:if>
     <xacro:if value="${arm_variant == 'follower'}">
-        <disable_collisions link1="${tf_prefix}${tf_prefix}camera_link" link2="${tf_prefix}camera_mount_d405" reason="Adjacent"/>
-        <disable_collisions link1="${tf_prefix}${tf_prefix}camera_mount_d405" link2="${tf_prefix}link_6" reason="Adjacent"/>
+        <disable_collisions link1="${tf_prefix}camera_link" link2="${tf_prefix}camera_mount_d405" reason="Adjacent"/>
+        <disable_collisions link1="${tf_prefix}camera_mount_d405" link2="${tf_prefix}link_6" reason="Adjacent"/>
     </xacro:if>  <!-- variant == 'follower' -->
 </robot>
